File: Cartes/TSAL/TSAL_Red/tsal_rouge maelle/carte.kicad_sch (KiCad schematic)
At the start: 17 parts

Commit message: tSAL ROUGE
Parts:
- V1: Spice_Model dc 5 pulse(0 70 1 0 0 3 6) -> dc 5 pulse(0 100 0 15 0 0 0)
Connections:
- net at CP1.1 (OUT), CP?.3 (IN-), R3.1: now also R6.2, TI1.8 (+VCC); no longer CP?.1 (OUT), R?.1, TI1.4 (RESET)
- net at CP1.5 (VCC+), CP?.5 (VCC+), R3.2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: no longer R6.2, TI1.8 (+VCC)
- new net: CP?.1 (OUT), R?.1, TI1.4 (RESET)
