File: Cartes/TSAL/TSAL_Green/TSAL_Green_1A/MAU/TSAL verte.kicad_sch (KiCad schematic)
At the start: 22 parts

Commit message: TSAL Fini
Parts:
- CP1, CP2: footprint SOT95P280X145-5N -> EPSA_lib:SOT95P280X145-5N; Render Name (none) -> Comparateur
- G1, G2, G6: footprint SOT95P280X145-5N -> EPSA_lib:SOT95P280X145-5N; Render Name (none) -> Gate AND
- G3, G5: footprint SOT95P280X145-5N -> EPSA_lib:SOT95P280X145-5N; Render Name (none) -> Gate NOR
- G4: footprint SOT95P280X145-5N -> EPSA_lib:SOT95P280X145-5N; Render Name (none) -> Gate OR
- G7, G8: footprint SOT95P280X145-5N -> EPSA_lib:SOT95P280X145-5N; Render Name (none) -> Gate XOR
- R1: footprint RESC3216X70N -> EPSA_lib:RESC3216X70N; Render Name (none) -> Résistance; Spice_Model 5750 -> 10
- R2: footprint RESC3216X70N -> EPSA_lib:RESC3216X70N; Render Name (none) -> Résistance; Spice_Model 250 -> 10
- R4, R5: footprint RESC3216X70N -> EPSA_lib:RESC3216X70N; Render Name (none) -> Résistance; Spice_Model 10k -> 10
