File: Cartes/TSAL/TSAL/TSAL.kicad_sch (KiCad schematic)
At the start: 61 parts, among them J1 2P Droit 2-11-2022, J10 2P Droit 2-11-2022, J11 2P Droit 2-11-2022, J2 2P Droit 2-11-2022, J3 2P Droit 2-11-2022, J4 3P Droit 22-11-2032, J5 2P Droit 2-11-2022, J6 2P Droit 2-11-2022, J7 2P Droit 2-11-2022, J8 2P Droit 2-11-2022, J9 2P Droit 2-11-2022, Q1 PMOS SI2343CDS-T1-GE3, Q2 NMOS SQ2348ES-T1_GE3, Q3 PMOS SI2343CDS-T1-GE3, Q4 NMOS SQ2348ES-T1_GE3

Commit message: TSAL Last update et percage
Parts:
- removed G8, G9: Gate AND SN74AHCT1G08DBVR, EPSA_lib:SOT95P280X145-5N, symbol EPSA_lib:Gate AND SN74AHCT1G08DBVR
- added G8, G9: Gate OR SN74AHCT1G32DBVR, EPSA_lib:SOT95P280X145-5N, symbol EPSA_lib:Gate OR SN74AHCT1G32DBVR
Connections:
- net +5V: now also G8.5 (VCC), G9.5 (VCC)
- net 0: now also G8.3 (GND), G9.3 (GND)
- net SCS log: now also G9.4 (Y)
- net at G5.4 (Y): now also G9.2 (B)
- net at G3.4 (Y): now also G8.1 (A)
- net at G4.4 (Y): now also G8.2 (B)
- new net: G8.4 (Y), G9.1 (A)

Commit message: Fin BSPD
Fin du BSPD et travail sur la TSAL
Parts:
- removed J5, J7, J8: 2P Droit 2-11-2022, EPSA_lib:MOLEX_22-11-2022, symbol EPSA_lib:2P Droit 2-11-2022
- removed R11, R13, R15, R16, R17, R18: Résistance RK73H2BLTDD2152F, EPSA_lib:RESC3216X70N, symbol EPSA_lib:Résistance RK73H2BLTDD2152F
- added J? (x3): 2P Droit 2-11-2022, EPSA_lib:MOLEX_22-11-2022, symbol EPSA_lib:2P Droit 2-11-2022
- added K? (x3): SSR CPC1394GR, EPSA_lib:CPC1394GR, symbol EPSA_lib:SSR CPC1394GR
- added R? (x6): Résistance RK73H2BLTDD2152F, EPSA_lib:RESC3216X70N, symbol EPSA_lib:Résistance RK73H2BLTDD2152F
Connections:
- net +5V: now also R14.2, R4.2, K?.3 (LOAD_1), K?.3 (LOAD_1), K?.3 (LOAD_1)
- net 0: now also DL1.10 (2~{PRE}), DL1.11 (2~{CLK}), DL1.12 (2D), DL1.13 (2~{CLR}), R?.2, R?.2, R?.2
- net Int AIR 1: now also K?.4 (LOAD_2), R?.1
- net Int AIR 2: now also K?.4 (LOAD_2), R?.1
- net Int PreCharge: now also K?.4 (LOAD_2), R?.1
- new net: K?.1 (+_CONTROL), R?.2 (x3)
- new net: J?.1, K?.2 (-_CONTROL) (x3)
- new net: J?.2, R?.1 (x3)
- no-connect marks 0 -> 3
Other:
- note added: "Green Connector Input"
- note added: "Green connector intentionnal input"
- note added: "power flag"
- note removed: "Green Connector"
- moved on the sheet: C5, C6, R23, R24, TI1

Commit message: Fin Cartes V2
Parts:
- removed G10, G6: Gate NAND SN74AHCT1G00DBVR, EPSA_lib:SOT95P280X145-5N, symbol EPSA_lib:Gate NAND SN74AHCT1G00DBVR
- removed G3, G4, G5: Gate XOR SN74AHCT1G86DBVR, EPSA_lib:SOT95P280X145-5N, symbol EPSA_lib:Gate XOR SN74AHCT1G86DBVR
- removed G9: Gate OR SN74AHCT1G32DBVR, EPSA_lib:SOT95P280X145-5N, symbol EPSA_lib:Gate OR SN74AHCT1G32DBVR
- removed Q1, Q3: PMOS SI2343CDS-T1-GE3, EPSA_lib:SOT95P237X112-3N, symbol EPSA_lib:PMOS SI2343CDS-T1-GE3
- removed R22: Résistance RK73H2BLTDD2152F, EPSA_lib:RESC3216X70N, symbol EPSA_lib:Résistance RK73H2BLTDD2152F
- added C10, C11, C12, C13, C14, C15, C17, C18, C19, C7, C8, C9: Condensateur 0805Y1000104JXT, EPSA_lib:CAPC2012X130N, symbol EPSA_lib:Condensateur 0805Y1000104JXT
- added D1, D10, D11, D2, D3, D4, D5, D6, D7, D8, D9: LED, LED_THT:LED_D5.0mm, symbol EPSA_lib:LED
- added G10, G11, G13: Gate OR SN74AHCT1G32DBVR, EPSA_lib:SOT95P280X145-5N, symbol EPSA_lib:Gate OR SN74AHCT1G32DBVR
- added G12: Gate NOR SN74AHCT1G02DBVR, EPSA_lib:SOT95P280X145-5N, symbol EPSA_lib:Gate NOR SN74AHCT1G02DBVR
- added G3, G4, G5, G6: Gate AND SN74AHCT1G08DBVR, EPSA_lib:SOT95P280X145-5N, symbol EPSA_lib:Gate AND SN74AHCT1G08DBVR
- added G9: Gate NAND SN74AHCT1G00DBVR, EPSA_lib:SOT95P280X145-5N, symbol EPSA_lib:Gate NAND SN74AHCT1G00DBVR
- added R11, R13, R15, R16: Résistance RK73H2BLTDD2152F, EPSA_lib:RESC3216X70N, symbol EPSA_lib:Résistance RK73H2BLTDD2152F
- added TP1, TP2, TP3, TP4: TestPoint, TestPoint:TestPoint_Pad_D2.0mm, symbol EPSA_lib:TestPoint
- R25, R26, R27: renamed from R?; Spice_Model 14k -> 500
- R3, R6, R9: Spice_Model 5k -> 500
- R8: Spice_Model 10 -> 500
- gave numbers to parts that had none: 9
Connections:
- net +12V: now also J10.1, J6.1
- net +5V: now also C10.2, C11.2, C12.2, C13.2, C14.2, C15.2, C17.2, C18.2, C19.2, C7.2, C8.2, C9.2, G10.5 (VCC), G11.5 (VCC), G12.5 (VCC), G13.5 (VCC), G3.5 (VCC), G4.5 (VCC), G5.5 (VCC), G6.5 (VCC), G9.5 (VCC)
- net 0: now also Q2.2, Q4.2, C10.1, C11.1, C12.1, C13.1, C14.1, C15.1, C17.1, C18.1, C19.1, C7.1, C8.1, C9.1, D1.1 (K), D10.1 (K), D11.1 (K), D2.1 (K), D3.1 (K), D4.1 (K), D5.1 (K), D6.1 (K), D7.1 (K), D8.1 (K), D9.1 (K), G10.3 (GND), G11.3 (GND), G12.3 (GND), G13.3 (GND), G3.3 (GND), G4.3 (GND), G5.3 (GND), G6.3 (GND), G9.3 (GND); no longer J1.1, J10.2, J2.1, J3.1, J6.2, R25.2, R26.2, R27.2, R8.1
- net AIR 1: now also G3.1 (A)
- net AIR 2: now also G4.1 (A)
- net CLR: now also TP1.1
- net Clign: now also Q4.1
- net DC-Link In: now also R16.2
- net Int AIR 1: now also G3.2 (B), G9.2 (B)
- net Int AIR 2: now also G10.1 (A), G4.2 (B)
- net Int PreCharge: now also G10.2 (B), G5.2 (B)
- net Lightning cond: now also G6.1 (A), R13.1
- net PRE: now also TP2.1
- net PreCharge: now also G5.1 (A)
- net SCS: now also R8.1, G6.2 (B)
- net SCS del: now also TP4.1
- net SCS log: now also G13.4 (Y), R15.1, TP3.1
- net VoltageAIR: now also G12.2 (B), R11.2
- net at Q2.1: now also G6.4 (Y)
- net at Q2.3: now also J6.2; no longer J6.1
- net at Q4.3: now also J10.2; no longer J10.1
- net at G8.1 (A): now also G3.4 (Y)
- net at R8.2: now also D2.2 (A); no longer Q2.2
- net at G8.4 (Y): now also G11.1 (A)
- net at G8.2 (B): now also G4.4 (Y)
- new net: D6.2 (A), R13.2
- new net: D11.2 (A), R27.2
- new net: D10.2 (A), R26.2
- new net: G12.4 (Y), G13.1 (A)
- new net: G11.4 (Y), G13.2 (B)
- new net: D1.2 (A), J1.1
- new net: G10.4 (Y), G9.1 (A)
- new net: G12.1 (A), G9.4 (Y)
- new net: D5.2 (A), R11.1
- new net: D8.2 (A), R16.1
- new net: D9.2 (A), R25.2
- new net: D7.2 (A), R15.2
- new net: D3.2 (A), J2.1
- new net: G11.2 (B), G5.4 (Y)
- new net: D4.2 (A), J3.1
Other:
- note added: "Em protection"
- note added: "Red act"
- note removed: "Red Push Pull"
- moved on the sheet: C1, C2, C3, C4, CP1, CP2, DL1, J10, J11, J6, J9, PS1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

Commit message: Cartes elec version cirly
Parts:
- added C16: C, Capacitor_THT:CP_Radial_D5.0mm_P2.00mm, symbol Device:C
- added R28, R29, R30: Résistance RK73H2BLTDD2152F, EPSA_lib:RESC3216X70N, symbol EPSA_lib:Résistance RK73H2BLTDD2152F
- R3, R6, R9: Spice_Model 500 -> 10k
- TI1: footprint EPSA_lib:SOIC127P600X175-8N -> Package_DIP:DIP-8_W7.62mm_Socket
Connections:
- net +12V: now also C16.2
- net +5V: now also R28.2, R29.2, R30.2
- net 0: now also J1.1, J2.1, J3.1, C16.1; no longer D1.1 (K), D3.1 (K), D4.1 (K)
- net AIR 1: now also D1.1 (K)
- net AIR 2: now also D3.1 (K)
- net PreCharge: now also D4.1 (K)
- net at D1.2 (A): now also R28.1; no longer J1.1
- net at D3.2 (A): now also R29.1; no longer J2.1
- net at D4.2 (A): now also R30.1; no longer J3.1
Other:
- note removed: "power flag"
- moved on the sheet: D1, D3, D4, R3, R6, R9
