File: Documentation/Kicad/Pack Elec/Kicad Spice Exemple/Comparateur Double Example.kicad_sch (KiCad schematic)
At the start: 9 parts

Commit message: Ajout du dongle SCS
Parts:
- CP1: footprint SOIC127P600X175-8N -> EPSA_lib:SOIC127P600X175-8N; Render Name (none) -> Comparateur Double
Changed lines of the file:
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@@
     (property "Reference" "CP1" (id 0) (at 149.86 77.47 0))
     (property "Value" "Comparateur Double LM393LVDR" (id 1) (at 149.86 80.01 0))
-    (property "Footprint" "SOIC127P600X175-8N" (id 2) (at 171.45 85.09 0)
+    (property "Footprint" "EPSA_lib:SOIC127P600X175-8N" (id 2) (at 171.45 85.09 0)
       (effects (font (size 1.27 1.27)) (justify left) hide)
     )
@@
     )
     (property "Spice_Lib_File" "${EPSA}\\SpiceModel\\CD_lm393.lib" (id 17) (at 149.86 82.55 0))
+    (property "Render Name" "Comparateur Double" (id 18) (at 149.86 83.82 0))
     (pin "1")
     (pin "2")
@@
     )
     (path "/1d7c6187-7d48-492c-a320-bbf515096f3c"
-      (reference "CP1") (unit 1) (value "Comparateur Double LM393LVDR") (footprint "SOIC127P600X175-8N")
+      (reference "CP1") (unit 1) (value "Comparateur Double LM393LVDR") (footprint "EPSA_lib:SOIC127P600X175-8N")
     )
     (path "/480bc776-2cf8-42bc-ae50-919e4eb824cb"
