File: Cartes/BENCH/Demonstrateur_VCU/TSAL.kicad_sch (KiCad schematic)
At the start: 99 parts, among them J16 2P Droit 2-11-2022, J17 2P Droit 2-11-2022, J18 2P Droit 2-11-2022, J19 3P Droit 22-11-2032, J20 2P Droit 2-11-2022, J21 2P Droit 2-11-2022, J22 2P Droit 2-11-2022, J23 2P Droit 2-11-2022, J24 2P Droit 2-11-2022, J25 2P Droit 2-11-2022, J26 2P Droit 2-11-2022, K10 SSR CPC1394GR, K11 SSR CPC1394GR, K12 SSR CPC1394GR, Q1 NMOS SQ2348ES-T1_GE3, Q2 NMOS SQ2348ES-T1_GE3

Commit message: ESF tentative
Parts:
- renumbered K10 to K11, K11 to K12, K12 to K13, R14 to R16, R15 to R17, R16 to R18, R17 to R19, R18 to R20, R19 to R21, R20 to R22, R21 to R23, R22 to R24, R23 to R25, R24 to R26, R25 to R27, R26 to R28, R27 to R29, R28 to R30, R29 to R31, R30 to R32, R31 to R33, R32 to R34, R33 to R35, R34 to R36, R35 to R37, R36 to R38, R37 to R39, R38 to R40, R39 to R41, R40 to R42, R41 to R43, R42 to R44, R43 to R45

Commit message: Ajout de l'AMS/IMD Reset
Parts:
- C10, C11, C12, C13, C2, C3, C4, C5, C6, C7, C8, C9: Spice_Model 10n -> (none); Spice_Netlist_Enabled Y -> (none); Spice_Primitive C -> (none)
- C15, C19: Spice_Model 1u -> (none); Spice_Netlist_Enabled Y -> (none); Spice_Primitive C -> (none)
- C16, C18: Spice_Model 2.2u -> (none); Spice_Netlist_Enabled Y -> (none); Spice_Primitive C -> (none)
- C17: Spice_Model 0.1u -> (none); Spice_Netlist_Enabled Y -> (none); Spice_Primitive C -> (none)
- C20: Spice_Model 0.01u -> (none); Spice_Netlist_Enabled Y -> (none); Spice_Primitive C -> (none)
- CP1: Spice_Lib_File ${EPSA}\SpiceModel\C_ts391.lib -> (none); Spice_Model TS391 -> (none); Spice_Netlist_Enabled Y -> (none); Spice_Node_Sequence 4,3,5,2,1 -> (none); Spice_Primitive X -> (none)
- CP2: Spice_Lib_File ${EPSA}\SpiceModel\CD_lm393.lib -> (none); Spice_Model LM2903B_Dual -> (none); Spice_Netlist_Enabled Y -> (none); Spice_Primitive X -> (none)
- D12, D13, D14, D15, D16, D17, D18, D19, D20, D21, D22: Spice_Model LED -> (none); Spice_Netlist_Enabled N -> (none); Spice_Primitive D -> (none)
- DL1: Spice_Lib_File ${EPSA}\SpiceModel\BD_SN74HCS72.lib -> (none); Spice_Model SN74HCS72_Double -> (none); Spice_Netlist_Enabled Y -> (none); Spice_Primitive X -> (none)
- G1, G13, G2, G3, G4, G5, G8: Spice_Lib_File ${EPSA}\SpiceModel\AND_SN74AHC1G08.lib -> (none); Spice_Model SN74AHC1G08 -> (none); Spice_Netlist_Enabled Y -> (none); Spice_Node_Sequence 4,1,2,5,3 -> (none); Spice_Primitive X -> (none)
- G10, G12, G7, G9: Spice_Lib_File ${EPSA}\SpiceModel\OR_SN74AHCT1G32.lib -> (none); Spice_Model SN74AHCT1G32 -> (none); Spice_Netlist_Enabled Y -> (none); Spice_Node_Sequence 4,1,2,5,3 -> (none); Spice_Primitive X -> (none)
- G11: Spice_Lib_File ${EPSA}\SpiceModel\NOR_SN74AHCT1G02.lib -> (none); Spice_Model SN74AHCT1G02 -> (none); Spice_Netlist_Enabled Y -> (none); Spice_Node_Sequence 4,1,2,5,3 -> (none); Spice_Primitive X -> (none)
- G6: Spice_Lib_File ${EPSA}\SpiceModel\NAND_SN74AHCT1G00.lib -> (none); Spice_Model SN74AHCT1G00 -> (none); Spice_Netlist_Enabled Y -> (none); Spice_Node_Sequence 4,1,2,5,3 -> (none); Spice_Primitive X -> (none)
- J16, J17, J18, J20, J21, J22, J23, J24, J25, J26: Spice_Model 22-11-2022 -> (none); Spice_Netlist_Enabled N -> (none); Spice_Primitive J -> (none)
- J19: Spice_Model 22-11-2032 -> (none); Spice_Netlist_Enabled N -> (none); Spice_Primitive J -> (none)
- K11, K12, K13: Spice_Lib_File ${EPSA}\SpiceModel\SSR.lib -> (none); Spice_Model SWITCH -> (none); Spice_Netlist_Enabled Y -> (none); Spice_Primitive X -> (none)
- PS1: Spice_Model Alim HP TSR_2-2450 -> (none); Spice_Netlist_Enabled N -> (none); Spice_Primitive R -> (none)
- Q1, Q2: Spice_Lib_File ${EPSA}\SpiceModel\NMOS_SQ2348ES_PS Rev A.LIB -> (none); Spice_Model SQ2348ES -> (none); Spice_Netlist_Enabled Y -> (none); Spice_Node_Sequence 3,1,2 -> (none); Spice_Primitive X -> (none)
- R16, R18, R20: Spice_Model 10k -> (none); Spice_Netlist_Enabled N -> (none); Spice_Primitive R -> (none)
- R17, R19, R21, R22, R24: Spice_Model 500 -> (none); Spice_Netlist_Enabled N -> (none); Spice_Primitive R -> (none)
- R23, R25, R28, R41, R42, R43: Spice_Model 500 -> (none); Spice_Netlist_Enabled Y -> (none); Spice_Primitive R -> (none)
- R26: Spice_Model 100k -> (none); Spice_Netlist_Enabled Y -> (none); Spice_Primitive R -> (none)
- R27: Spice_Model 50k -> (none); Spice_Netlist_Enabled Y -> (none); Spice_Primitive R -> (none)
- R29, R38, R39, R40: Spice_Model 10k -> (none); Spice_Netlist_Enabled Y -> (none); Spice_Primitive R -> (none)
- R30, R37: Spice_Model 500k -> (none); Spice_Netlist_Enabled Y -> (none); Spice_Primitive R -> (none)
- R31, R36: Spice_Model 600k -> (none); Spice_Netlist_Enabled Y -> (none); Spice_Primitive R -> (none)
- R32, R35: Spice_Model 5k -> (none); Spice_Netlist_Enabled Y -> (none); Spice_Primitive R -> (none)
- R33, R34: Spice_Model 390k -> (none); Spice_Netlist_Enabled Y -> (none); Spice_Primitive R -> (none)
- R44: Spice_Model 2k -> (none); Spice_Netlist_Enabled Y -> (none); Spice_Primitive R -> (none)
- R45: Spice_Model 200k -> (none); Spice_Netlist_Enabled Y -> (none); Spice_Primitive R -> (none)
- RV1: Spice_Lib_File ${EPSA}\SpiceModel\VARYSTOR.lib -> (none); Spice_Model VARYSTOR Rtot=20k Part=0.78 -> (none); Spice_Netlist_Enabled Y -> (none); Spice_Primitive X -> (none)
- TI1: Spice_Lib_File ${EPSA}\SpiceModel\555_TLC555.lib -> (none); Spice_Model TLC555 -> (none); Spice_Netlist_Enabled Y -> (none); Spice_Node_Sequence 6,5,2,4,3,7,8,1 -> (none); Spice_Primitive X -> (none)
- TP1, TP2, TP3, TP4: value TestPoint -> ${SIM.PARAMS}; Spice_Netlist_Enabled N -> (none); Spice_Primitive R -> (none)
