File: Cartes/AMS & IMD Reset/AMS & IMD Reset.kicad_sch (KiCad schematic)
At the start: 10 parts, among them J1 3P Droit 22-11-2032, J2 3P Droit 22-11-2032, J3 2P Droit 2-11-2022, J4 2P Droit 2-11-2022, K1 SSR CPC1394GR, K2 V23079-B1203-B301, U1 Alim LP TSR_0.5-2450

Commit message: Maj cartes
Parts:
- C1: value Condensateur 0805Y1000104JXT -> 10u
- R1: value Résistance RK73H2BLTDD2152F -> 2k2
Changed lines of the file:
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@@
   )
   (symbol (lib_id "EPSA_lib:Condensateur 0805Y1000104JXT") (at 227.33 149.86 0) (unit 1)
-    (in_bom yes) (on_board yes) (dnp no) (fields_autoplaced)
+    (in_bom yes) (on_board yes) (dnp no)
     (property "Reference" "C1" (at 233.68 143.51 0)
       (effects (font (size 1.27 1.27)))
     )
-    (property "Value" "Condensateur 0805Y1000104JXT" (at 247.65 147.32 0)
-      (effects (font (size 1.27 1.27)) (justify left) hide)
+    (property "Value" "10u" (at 236.22 152.4 0)
+      (effects (font (size 1.27 1.27)) (justify left))
     )
     (property "Footprint" "EPSA_lib:CAPC2012X130N" (at 247.65 149.86 0)
@@
       (effects (font (size 1.27 1.27)) (justify left) hide)
     )
-    (property "Sim.Pins" "1=1 2=2" (at 227.33 149.86 0)
-      (effects (font (size 1.27 1.27)) hide)
-    )
-    (property "Sim.Device" "SPICE" (at 247.65 144.78 0)
+    (property "Sim.Pins" "1=+ 2=-" (at 227.33 149.86 0)
+      (effects (font (size 1.27 1.27)) hide)
+    )
+    (property "Sim.Device" "C" (at 247.65 144.78 0)
       (effects (font (size 1.27 1.27)) (justify left) hide)
     )
@@
   )
   (symbol (lib_id "EPSA_lib:Résistance RK73H2BLTDD2152F") (at 171.45 64.77 0) (unit 1)
-    (in_bom yes) (on_board yes) (dnp no) (fields_autoplaced)
+    (in_bom yes) (on_board yes) (dnp no)
     (property "Reference" "R1" (at 180.34 59.69 0)
       (effects (font (size 1.27 1.27)))
     )
-    (property "Value" "Résistance RK73H2BLTDD2152F" (at 196.85 62.23 0)
-      (effects (font (size 1.27 1.27)) (justify left) hide)
+    (property "Value" "2k2" (at 179.07 64.77 0)
+      (effects (font (size 1.27 1.27)) (justify left))
     )
     (property "Footprint" "EPSA_lib:RESC3216X70N" (at 196.85 64.77 0)
@@
       (effects (font (size 1.27 1.27)) (justify left) hide)
     )
-    (property "Sim.Pins" "1=1 2=2" (at 171.45 64.77 0)
-      (effects (font (size 1.27 1.27)) hide)
-    )
-    (property "Sim.Device" "SPICE" (at 196.85 59.69 0)
-      (effects (font (size 1.27 1.27)) (justify left) hide)
-    )
+    (property "Sim.Pins" "1=+ 2=-" (at 171.45 64.77 0)
+      (effects (font (size 1.27 1.27)) hide)
+    )
+    (property "Sim.Device" "R" (at 196.85 59.69 0)
+      (effects (font (size 1.27 1.27)) (justify left) hide)
+    )
