File: Cartes/BENCH/Demonstrateur_VCU/Carte_VCU/Carte_VCU - Back.kicad_sch (KiCad schematic)
At the start: 46 parts, among them J1 Conn_01x02_Female, J10 Conn_01x02_Female, J11 Conn_01x02_Female, J12 Conn_01x04_Female, J13 Conn_01x03_Female, J14 Conn_01x03_Female, J15 Conn_01x03_Female, J2 Conn_01x02_Female, J3 Conn_01x02_Female, J4 Conn_01x02_Female, J5 Conn_01x02_Female, J6 Conn_01x02_Female, J7 Conn_01x02_Female, J8 Conn_01x03_Female, J9 Conn_01x03_Female, SW1 SW_Push_SPDT, SW2 SW_Push_SPDT, SW3 SW_Push_SPDT, SW4 SW_Push_SPDT, SW5 SW_MEC_5G, SW6 SW_Push_SPDT, SW7 SW_Push_SPDT, SW8 SW_Push_SPDT, SW9 SW_Push_SPDT

Commit message: Rebase
Parts:
- R10, R11, R12, R13, R14, R15, R5, R6, R7, R8, R9: Spice_Model (none) -> 5k; Spice_Netlist_Enabled (none) -> Y; Spice_Primitive (none) -> R
