File: 02 - Documentation/BASTIE/Cartes Valkyriz/BMS/BMS V1.0/BMS V1.0.kicad_sch (KiCad schematic)
At the start: 31 parts, among them IC1 LT3990EMSE#TRPBF, IC2 LTC6255IS6#TRMPBF, IC3 ADG728BRUZ-REEL7, IC4 ADG728BRUZ-REEL7, IC6 LTC6811IG-1#PBF, J1 Conn_01x02_Pin, J3 Conn_01x02_Pin, T1 SM91501ALE

Commit message: Import BMS files
Import des fichiers BMS directement depuis le git d'eymeric
Parts:
- added C12, C13, C14, C15, C16, C17, C18, C19, C20, C21, C22, C23, C24: 10n, Capacitor_SMD:C_0805_2012Metric_Pad1.18x1.45mm_HandSolder, symbol Device:C
- added C25: 100n, Capacitor_SMD:C_0805_2012Metric_Pad1.18x1.45mm_HandSolder, symbol Device:C
- added C26: 1u, Capacitor_SMD:C_0805_2012Metric_Pad1.18x1.45mm_HandSolder, symbol Device:C
- added J2, J6: Conn_01x07_Pin, EPSA:SHDRRA7W77P0X254_1X7_2032X1359X699P, symbol Connector:Conn_01x07_Pin
- added J4, J5: Conn_01x08_Pin, EPSA:SHDRRA9W69P0X254_1X9_2527X1359X741P, symbol Connector:Conn_01x09_Pin
- added Q1, Q10, Q11, Q12, Q2, Q3, Q4, Q5, Q6, Q7, Q8, Q9: Q_PMOS_GDS, EPSA:SOT-23-3, symbol Device:Q_PMOS_GSD
- added R12, R18, R21, R24, R27, R30, R33, R36, R39, R42, R45, R48: 3.3K, Resistor_SMD:R_1206_3216Metric_Pad1.30x1.75mm_HandSolder, symbol Device:R
- added R13, R15, R17, R20, R23, R26, R29, R32, R35, R38, R41, R44, R47, R51: 100, Resistor_SMD:R_1206_3216Metric_Pad1.30x1.75mm_HandSolder, symbol Device:R
- added R14, R16, R19, R22, R25, R28, R31, R34, R37, R40, R43, R46: 25, Resistor_SMD:R_2512_6332Metric_Pad1.40x3.35mm_HandSolder, symbol Device:R
- added R49, R50: 1k, Resistor_SMD:R_1206_3216Metric_Pad1.30x1.75mm_HandSolder, symbol Device:R
- added R52: 10k, Resistor_SMD:R_1206_3216Metric_Pad1.30x1.75mm_HandSolder, symbol Device:R
- C1, C10, C11, C2, C3, C4, C5, C6, C7, C8, C9: footprint (none) -> Capacitor_SMD:C_0805_2012Metric_Pad1.18x1.45mm_HandSolder
- IC1: footprint SOP50P490X110-17N -> EPSA:SOP50P490X110-17N
- IC2: footprint SOT95P280X100-6N -> EPSA:SOT95P280X100-6N
- IC3, IC4: footprint SOP65P640X120-16N -> EPSA:SOP65P640X120-16N
- IC6: footprint SOP50P780X200-48N -> EPSA:SOP50P780X200-48N
- J1, J3: footprint (none) -> EPSA:RHDR2W97P0X254_1X2_654X508X1379P
- L1: footprint (none) -> Inductor_SMD:L_1210_3225Metric_Pad1.42x2.65mm_HandSolder
- R1, R2, R3, R4, R5, R6, R7: footprint (none) -> Resistor_SMD:R_1206_3216Metric_Pad1.30x1.75mm_HandSolder
- R10: renamed from R11; footprint (none) -> Resistor_SMD:R_1206_3216Metric_Pad1.30x1.75mm_HandSolder
- R11: renamed from R10; footprint (none) -> Resistor_SMD:R_1206_3216Metric_Pad1.30x1.75mm_HandSolder
- R8: renamed from R9; footprint (none) -> Resistor_SMD:R_1206_3216Metric_Pad1.30x1.75mm_HandSolder
- R9: renamed from R8; footprint (none) -> Resistor_SMD:R_1206_3216Metric_Pad1.30x1.75mm_HandSolder
- T1: footprint SOP200P1473X500-12N -> EPSA:SOP200P1473X500-12N
Connections:
- net GND is gone; now on net -VDC: C2.1, C4.1, IC1.17 (GND_2), IC1.8 (GND_1), R1.2, R3.2
- net +5V: now also C26.1; no longer IC1.4 (EN/UVLO)
- net +BATT: now also J2.2 (Pin_2), Q11.2 (S), R44.1, R51.1
- net -VDC: now also IC6.36 (DTEN), C24.2, C25.2, C26.2, J2.1 (Pin_1), J4.1 (Pin_1), J5.9 (Pin_9), J6.7 (Pin_7), R46.1, R47.1, R50.2
- net IMA: now also R10.1, T1.12 (SEC1_3); no longer R8.1, T1.7 (SEC2_1)
- net IMB: now also R9.2, T1.9 (SEC2_3); no longer R11.2, T1.10 (SEC1_1)
- net IPA: now also R11.2, T1.10 (SEC1_1); no longer R9.2, T1.9 (SEC2_3)
- net IPB: now also R8.1, T1.7 (SEC2_1); no longer R10.1, T1.12 (SEC1_3)
- net T1: now also J4.9 (Pin_9)
- net T10: now also J5.7 (Pin_7)
- net T11: now also J5.6 (Pin_6)
- net T12: now also J5.5 (Pin_5)
- net T13: now also J5.4 (Pin_4)
- net T14: now also J5.3 (Pin_3)
- net T15: now also J5.2 (Pin_2)
- net T16: now also J5.1 (Pin_1)
- net T2: now also J4.8 (Pin_8)
- net T3: now also J4.7 (Pin_7)
- net T4: now also J4.6 (Pin_6)
- net T5: now also J4.5 (Pin_5)
- net T6: now also J4.4 (Pin_4)
- net T7: now also J4.3 (Pin_3)
- net T8: now also J4.2 (Pin_2)
- net T9: now also J5.8 (Pin_8)
- net at IC2.3 (+IN), IC3.8 (D), IC4.8 (D): now also R52.2
- net VREF2: now reaches C10.1, IC6.34 (VREF2)
- net VREF2: now also R52.1
- net at IC6.1 (V+): now also C25.1, R51.2
- net C8: now reaches IC6.10 (C8)
- net C8: now also C18.1, C19.2, R32.2
- net S8: now reaches IC6.11 (S8)
- net S8: now also R33.2
- net C7: now reaches IC6.12 (C7)
- net C7: now also C17.1, C18.2, R29.2
- net S7: now reaches IC6.13 (S7)
- net S7: now also R30.2
- net C6: now reaches IC6.14 (C6)
- net C6: now also C16.1, C17.2, R26.2
- net S6: now reaches IC6.15 (S6)
- net S6: now also R27.2
- net C5: now reaches IC6.16 (C5)
- net C5: now also C15.1, C16.2, R23.2
- net S5: now reaches IC6.17 (S5)
- net S5: now also R24.2
- net C4: now reaches IC6.18 (C4)
- net C4: now also C14.1, C15.2, R20.2
- net S4: now reaches IC6.19 (S4)
- net S4: now also R21.2
- net C12: now reaches IC6.2 (C12)
- net C12: now also C22.1, R44.2
- net C3: now reaches IC6.20 (C3)
- net C3: now also C13.1, C14.2, R17.2
- net S3: now reaches IC6.21 (S3)
- net S3: now also R18.2
- net C2: now reaches IC6.22 (C2)
- net C2: now also C12.1, C13.2, R13.2
- net S2: now reaches IC6.23 (S2)
- net S2: now also R12.2
- net C1: now reaches IC6.24 (C1)
- net C1: now also C12.2, C23.1, R15.2
- net S1: now reaches IC6.25 (S1)
- net S1: now also R48.2
- net C0: now reaches IC6.26 (C0)
- net C0: now also C23.2, C24.1, R47.2
- net S12: now reaches IC6.3 (S12)
- net S12: now also R45.2
- net Enable: now reaches IC6.38 (DRIVE)
- net Enable: now also IC1.4 (EN/UVLO)
- net C11: now reaches IC6.4 (C11)
- net C11: now also C21.1, C22.2, R41.2
- net at IC6.45 (IBIAS): now also R49.1
- net at IC6.46 (ICMP): now also R49.2, R50.1
- net S11: now reaches IC6.5 (S11)
- net S11: now also R42.2
- net C10: now reaches IC6.6 (C10)
- net C10: now also C20.1, C21.2, R38.2
- net S10: now reaches IC6.7 (S10)
- net S10: now also R39.2
- net C9: now reaches IC6.8 (C9)
- net C9: now also C19.1, C20.2, R35.2
- net S9: now reaches IC6.9 (S9)
- net S9: now also R36.2
- new net: Q6.1 (G), R30.1
- new net: Q6.3 (D), R28.2
- new net: Q5.3 (D), R25.2
- new net: Q4.1 (G), R24.1
- new net: Q12.1 (G), R48.1
- new net: Q11.1 (G), R45.1
- new net: Q1.1 (G), R12.1
- new net: Q1.3 (D), R14.2
- new net: Q4.3 (D), R22.2
- new net: Q3.1 (G), R21.1
- new net: Q8.3 (D), R34.2
- new net: Q10.1 (G), R42.1
- new net: Q8.1 (G), R36.1
- new net: Q5.1 (G), R27.1
- new net: Q7.1 (G), R33.1
- new net: Q7.3 (D), R31.2
- new net: Q9.3 (D), R37.2
- new net: Q10.3 (D), R40.2
- new net: Q11.3 (D), R43.2
- new net: Q3.3 (D), R19.2
- new net: Q12.3 (D), R46.2
- new net: Q2.1 (G), R18.1
- new net: Q2.3 (D), R16.2
- new net: Q9.1 (G), R39.1
- new net Cell 1: J6.6 (Pin_6), Q12.2 (S), R14.1, R15.1
- new net Cell 10: J2.3 (Pin_3), Q9.2 (S), R38.1, R40.1
- new net Cell 11: J6.1 (Pin_1), Q10.2 (S), R41.1, R43.1
- new net Cell 2: J2.7 (Pin_7), Q1.2 (S), R13.1, R16.1
- new net Cell 3: J6.5 (Pin_5), Q2.2 (S), R17.1, R19.1
- new net Cell 4: J2.6 (Pin_6), Q3.2 (S), R20.1, R22.1
- new net Cell 5: J6.4 (Pin_4), Q4.2 (S), R23.1, R25.1
- new net Cell 6: J2.5 (Pin_5), Q5.2 (S), R26.1, R28.1
- new net Cell 7: J6.3 (Pin_3), Q6.2 (S), R29.1, R31.1
- new net Cell 8: J2.4 (Pin_4), Q7.2 (S), R32.1, R34.1
- new net Cell 9: J6.2 (Pin_2), Q8.2 (S), R35.1, R37.1
- no-connect marks 13 -> 15
Other:
- note added: "5-103635-6"
- note added: "5-103635-7"
- note added: "Balancing"
- note added: "LTC6811"
- note added: "PM1210-330J-RC"
- note added: "PMOS BSS315P H6327"
- moved on the sheet: C10, C11, C6, C7, C8, C9, IC6, J1, J3, R10, R11, R8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
