File: 02 - Documentation/BASTIE/Cartes Valkyriz/TSAL/TSAL_pack/TSAL.kicad_pcb (KiCad board)
At the start: 2 copper layers, 58 x 58 mm, 122 parts, among them J1 2P Droit 2-11-2022, J2 2P Droit 2-11-2022, J3 2P Droit 2-11-2022, J4 3P Droit 22-11-2032, J5 2P Droit 2-11-2022, J6 2P Droit 2-11-2022, J7 4P Droit 22-11-2042, J8 3P Droit 22-11-2032, J9 2P Droit 2-11-2022, Q1 NMOS SQ2348ES-T1_GE3, Q2 NMOS SQ2348ES-T1_GE3, Q3 PMOS SI2343CDS-T1-GE3, Q4 PMOS SI2343CDS-T1-GE3, U1 Opamp_Quad, U2 Opamp

Commit message: Un peu plus d'élec
Other:
- board text removed: "EPSA"
Changed lines of the file:
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@@
     (pad "3" smd roundrect (at 1.1375 0) (size 1.325 0.6) (layers "F.Cu" "F.Paste" "F.Mask") (roundrect_rratio 0.25)
       (net 68 "Net-(Q3-Pad3)") (pintype "passive"))
-    (model "${KICAD6_3DMODEL_DIR}/Package_TO_SOT_SMD.3dshapes/SOT-23-3.wrl"
+    (model "${KICAD7_3DMODEL_DIR}/Package_TO_SOT_SMD.3dshapes/SOT-23.step"
       (offset (xyz 0 0 0))
       (scale (xyz 1 1 1))
@@
     (pad "3" smd roundrect (at 1.1375 0) (size 1.325 0.6) (layers "F.Cu" "F.Paste" "F.Mask") (roundrect_rratio 0.25)
       (net 68 "Net-(Q3-Pad3)") (pintype "passive"))
-    (model "${KICAD6_3DMODEL_DIR}/Package_TO_SOT_SMD.3dshapes/SOT-23-3.wrl"
+    (model "${KICAD7_3DMODEL_DIR}/Package_TO_SOT_SMD.3dshapes/SOT-23.step"
       (offset (xyz 0 0 0))
       (scale (xyz 1 1 1))
@@
   (gr_arc (start 98.75 30.25) (mid 99.921573 27.421573) (end 102.75 26.25)
     (stroke (width 0.1) (type default)) (layer "Edge.Cuts"))
-  (gr_text "EPSA" (at 149.225 64.897) (layer "F.SilkS")
-    (effects (font (size 0.8 0.8) (thickness 0.15)) (justify left bottom))
-  )
   (gr_text "DCi" (at 138.303 52.705) (layer "F.SilkS")
     (effects (font (size 0.7 0.7) (thickness 0.14) bold))
