File: 02 - Documentation/BASTIE/Cartes Artemiz/Inverter_Voltage Sensor/Inverter_Voltage Sensor.kicad_sch (KiCad schematic)
At the start: 18 parts, among them J1 3P Droit 22-11-2032, K1 SSR CPC1394GR

Commit message: Maj Cartes
Parts:
- added R13, R14: 8k2, EPSA_lib:RESC3216X70N, symbol EPSA_lib:Résistance RK73H2BLTDD2152F
- added R15: 3k9, EPSA_lib:RESC3216X70N, symbol EPSA_lib:Résistance RK73H2BLTDD2152F
Connections:
- net +5VA: now also R13.2
- net Exit: now also R13.1, R14.2, R15.2; no longer K1.3 (LOAD_1), R7.2
- net GND: now also R14.1
- new net Raw_Exit: K1.3 (LOAD_1), R15.1, R7.2
Other:
- note added: "SCS"
