File: 02 - Documentation/BASTIE/Cartes Artemiz/VCU_Bis/VCU_Bis.kicad_sch (KiCad schematic)
At the start: 18 parts, among them J1 4P Droit 22-11-2042, J2 4P Droit 22-11-2042, J3 4P Droit 22-11-2042, J4 2P Droit 2-11-2022, U1 Alim LP TSR_0.5-2450

Commit message: Reset + EPSA_lib
Parts:
- removed R11: 820, EPSA_lib:RESC3216X70N, symbol EPSA_lib:Résistance RK73H2BLTDD2152F
- removed R12: 390, EPSA_lib:RESC3216X70N, symbol EPSA_lib:Résistance RK73H2BLTDD2152F
- added R2, R3: 8k2, EPSA_lib:RESC3216X70N, symbol EPSA_lib:Résistance RK73H2BLTDD2152F
- R10, R4, R7: value 820 -> 3k9
- R13, R14, R5, R8: value 820 -> 8k2
- R15: value 390 -> 3k9
- R6, R9: value 390 -> 8k2
Connections:
- net +5V: now also R5.2, R8.2, R2.2; no longer R10.2, R4.2, R7.2
- net GND: now also R6.1, R9.1, R3.1; no longer R5.1, R8.1
- net Int AIR+: now also R4.2, R2.1, R3.2; no longer R10.1
- net Int Dis: now also R5.1, R6.2, R7.2; no longer R7.1, R8.2, R9.2
- net Int Pre: now also R10.2, R8.1, R9.2; no longer R4.1, R5.2, R6.2
- net Int VCU AIR+: now also R4.1
- net Int VCU Dis: now also R7.1; no longer R9.1
- net Int VCU Pre: now also R10.1; no longer R6.1

Commit message: Encore qlq corrections
Parts:
- removed J2: 4P Droit 22-11-2042, EPSA_lib:MOLEX_22-11-2042, symbol EPSA_lib:4P Droit 22-11-2042
- removed R1: 120, EPSA_lib:RESC3216X70N, symbol EPSA_lib:Résistance RK73H2BLTDD2152F
- added C1: C, Capacitor_THT:CP_Radial_D5.0mm_P2.00mm, symbol Device:C
- added C2: 10n, EPSA_lib:CAPC2012X130N, symbol EPSA_lib:Condensateur 0805Y1000104JXT
Connections:
- net +12V: now also C1.1
- net +5V: now also C2.1
- net GND: now also C1.2, C2.2
