File: 02 - Documentation/MODAC/Cartes Elec/AIR Controller/Discharge Controller.kicad_sch (KiCad schematic)
At the start: 23 parts, among them J1 3P Droit 22-11-2032, J4 2P Droit 2-11-2022, K2 Relais PCB, Q1 NMOS SQ2348ES-T1_GE3, U1 Alim LP TSR_0.5-2450, U4 Opamp_Dual, U5 ${SIM.PARAMS}

Commit message: MAJ 3D Modac
Parts:
- removed G2: Gate AND SN74AHCT1G08DBVR, EPSA_lib:SOT95P280X145-5N, symbol EPSA_lib:Gate AND SN74AHCT1G08DBVR
- added PorteNAND1: Gate NAND SN74AHCT1G00DBVR, EPSA_lib:SOT95P280X145-5N, symbol EPSA_lib:Gate NAND SN74AHCT1G00DBVR
- U4: symbol EPSA_Lib:Comparator_Dual -> EPSA_lib:Comparator_Dual
- U5: symbol EPSA_lib:Opamp -> EPSA_Lib:Opamp
Connections:
- net +5V: now also PorteNAND1.5 (VCC)
- net GND: now also PorteNAND1.3 (GND)
- net Raw_Relay_Closed: now also J1.1, V3.1 (E1)
- net Relay_Closed: now also PorteNAND1.1, PorteNAND1.2
- net SC in: now also J1.2; no longer J1.1
- net at G1.1: now also PorteNAND1.4
- removed net Raw_Relay_On: J1.2, V3.1 (E1)
Other:
- note added: "Controlling a NC Relay"
- note removed: "Controlling a NO Relay"
