File: 02 - Documentation/MODAC/Cartes Elec/AMS_IMD_Reset (Charger)/AMS_IMD_Reset.kicad_sch (KiCad schematic)
At the start: 53 parts, among them J1 2P Droit 2-11-2022, J2 2P Droit 2-11-2022, J3 2P Droit 2-11-2022, J4 2P Droit 2-11-2022, J5 2P Droit 2-11-2022, J6 2P Droit 2-11-2022, J7 4P Droit 22-11-2042, K1 Relais PCB, K2 Bistable V23079B1201B301, K3 Relais PCB, K4 Bistable V23079B1201B301, Q1 NMOS SQ2348ES-T1_GE3, Q2 NMOS SQ2348ES-T1_GE3, Q3 NMOS SQ2348ES-T1_GE3, Q4 NMOS SQ2348ES-T1_GE3, Q5 NMOS SQ2348ES-T1_GE3, Q6 NMOS SQ2348ES-T1_GE3, Q7 NMOS SQ2348ES-T1_GE3, Q8 NMOS SQ2348ES-T1_GE3, U1 Alim LP TSR_0.5-2450, U2 ${SIM.PARAMS}

Commit message: MAJ modèles 3D KICAD
Parts:
- added J8: 2P Droit 2-11-2022, EPSA_lib:MOLEX_22-11-2022, symbol EPSA_Lib:2P Droit 2-11-2022
Connections:
- net GND: now also J6.2, J8.1
- net at Q8.3, R14.2: now also J8.2; no longer J6.1
- net at Q7.3, R13.2: now also J6.1; no longer J6.2
Other:
- moved on the sheet: J6

Commit message: Prise en compte retours JDL
Parts:
- added R19, R20, R21, R22: 1k, EPSA_lib:RESC3216X70N, symbol EPSA_Lib:Résistance RK73H2BLTDD2152F
Connections:
- net SC_Closed_AMS: now also R19.1, R21.1; no longer Q6.1, Q8.1
- net SC_Closed_IMD: now also R20.1, R22.1; no longer Q5.1, Q7.1
- new net: Q8.1, R19.2
- new net: Q6.1, R21.2
- new net: Q5.1, R22.2
- new net: Q7.1, R20.2
Other:
- moved on the sheet: J6, J8, K1, K3, Q5, Q6, Q7, Q8, R13, R14
