File: 02 - Documentation/BASTIE/Cartes Artemiz/TSAL (version SCS output)/TSAL/TSAL.kicad_pcb (KiCad board)
At the start: 2 copper layers, 58 x 58 mm, 127 parts, among them J1 2P Droit 2-11-2022, J2 2P Droit 2-11-2022, J3 2P Droit 2-11-2022, J4 3P Droit 22-11-2032, J5 2P Droit 2-11-2022, J6 2P Droit 2-11-2022, J7 4P Droit 22-11-2042, J8 3P Droit 22-11-2032, J9 2P Droit 2-11-2022, Q3 PMOS SI2343CDS-T1-GE3, Q4 PMOS SI2343CDS-T1-GE3, U1 Opamp_Quad, U2 Opamp

Commit message: Aop fixes
Connections:
- U2 pad 2: /VoltageAIR -> GND
- U2 pad 4: +5V -> /VoltageAIR
- U2 pad 5: GND -> +5V
Routing:
- net /VoltageAIR: track 69.8 -> 72.4 mm
- net GND: track 111.2 -> 113.5 mm
- net +5V: track 412.3 -> 411.5 mm
