File: 02 - Documentation/BASTIE/Cartes Artemiz/JLCPCB-ver/SCS Red Led/SCS Red Led.kicad_pcb (KiCad board)
At the start: 2 copper layers, 30.7 x 29 mm, 17 parts, among them J1 Conn_01x02, J2 Conn_01x02, U1 74AHC1G08, U4 CPC1017N, U5 LMV321IDBVR, U6 78L05G, U7 LMV321IDBVR, U8 LMV321IDBVR

Commit message: corrections jlcp ver cartes
Connections:
- U5 pad 1: Net-(U5-+) -> /PCB_State_OK
- U7 pad 3: Net-(U5-+) -> /PCB_State_OK
- U7 pad 4: Net-(U5-+) -> /PCB_State_OK
- U8 pad 3: Net-(U5-+) -> /PCB_State_OK
Routing:
- net /PCB_State_OK: track 0.00 -> 58.0 mm
- net Net-(U5-+): track 46.7 -> 0.00 mm
Changed lines of the file:
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@@
 	(net 10 "/SCS_Compliance")
 	(net 11 "/PCB_State_OK")
-	(net 12 "Net-(U5-+)")
 	(footprint "PCM_JLCPCB:C_0805"
 		(layer "F.Cu")
@@
 			(layers "F.Cu" "F.Mask" "F.Paste")
 			(roundrect_rratio 0.25)
-			(net 12 "Net-(U5-+)")
+			(net 11 "/PCB_State_OK")
 			(pinfunction "-")
 			(pintype "input")
@@
 			(layers "F.Cu" "F.Mask" "F.Paste")
 			(roundrect_rratio 0.25)
-			(net 12 "Net-(U5-+)")
+			(net 11 "/PCB_State_OK")
 			(pinfunction "OUT")
 			(pintype "output")
@@
 			(layers "F.Cu" "F.Mask" "F.Paste")
 			(roundrect_rratio 0.25)
-			(net 12 "Net-(U5-+)")
+			(net 11 "/PCB_State_OK")
 			(pinfunction "-")
 			(pintype "input")
@@
 			(layers "F.Cu" "F.Mask" "F.Paste")
 			(roundrect_rratio 0.25)
-			(net 12 "Net-(U5-+)")
+			(net 11 "/PCB_State_OK")
 			(pinfunction "+")
 			(pintype "input")
@@
 		(width 0.2)
 		(layer "F.Cu")
-		(net 12)
+		(net 11)
 	)
 	(segment
@@
 		(width 0.2)
 		(layer "F.Cu")
-		(net 12)
+		(net 11)
 	)
 	(segment
@@
 		(width 0.2)
 		(layer "F.Cu")
-		(net 12)
+		(net 11)
 	)
 	(segment
@@
 		(width 0.2)
 		(layer "F.Cu")
-		(net 12)
+		(net 11)
 	)
 	(segment
@@
 		(width 0.2)
 		(layer "F.Cu")
-		(net 12)
+		(net 11)
+	)
+	(segment
+		(start 76.642 75.8245)
+		(end 77.813 74.6535)
+		(width 0.2)
+		(layer "F.Cu")
+		(net 11)
 	)
 	(segment
@@
 		(width 0.2)
 		(layer "F.Cu")
-		(net 12)
+		(net 11)
 	)
 	(segment
@@
 		(width 0.2)
 		(layer "F.Cu")
-		(net 12)
+		(net 11)
 	)
 	(segment
@@
 		(width 0.2)
 		(layer "F.Cu")
-		(net 12)
+		(net 11)
 	)
 	(segment
@@
 		(width 0.2)
 		(layer "F.Cu")
-		(net 12)
+		(net 11)
 	)
 	(segment
@@
 		(width 0.2)
 		(layer "F.Cu")
-		(net 12)
+		(net 11)
+	)
+	(segment
+		(start 77.813 69.123032)
+		(end 76.854968 68.165)
+		(width 0.2)
+		(layer "F.Cu")
+		(net 11)
 	)
 	(segment
@@
 		(width 0.2)
 		(layer "F.Cu")
-		(net 12)
+		(net 11)
 	)
 	(segment
@@
 		(width 0.2)
 		(layer "F.Cu")
-		(net 12)
+		(net 11)
 	)
 	(segment
@@
 		(width 0.2)
 		(layer "F.Cu")
-		(net 12)
+		(net 11)
 	)
 	(segment
@@
 		(width 0.2)
 		(layer "F.Cu")
-		(net 12)
+		(net 11)
 	)
 	(segment
@@
 		(width 0.2)
 		(layer "F.Cu")
-		(net 12)
+		(net 11)
+	)
+	(segment
+		(start 75.512999 68.165)
+		(end 74.911999 67.564)
+		(width 0.2)
+		(layer "F.Cu")
+		(net 11)
 	)
 	(segment
@@
 		(width 0.2)
 		(layer "F.Cu")
-		(net 12)
+		(net 11)
 	)
 	(segment
@@
 		(width 0.2)
 		(layer "F.Cu")
-		(net 12)
+		(net 11)
 	)
 	(segment
@@
 		(width 0.2)
 		(layer "F.Cu")
-		(net 12)
+		(net 11)
 	)
 	(segment
@@
 		(width 0.2)
 		(layer "F.Cu")
-		(net 12)
+		(net 11)
 	)
 	(segment
@@
 		(width 0.2)
 		(layer "F.Cu")
-		(net 12)
+		(net 11)
 	)
 	(segment
@@
 		(width 0.2)
 		(layer "F.Cu")
-		(net 12)
+		(net 11)
 	)
 	(segment
@@
 		(width 0.2)
 		(layer "F.Cu")
-		(net 12)
+		(net 11)
 	)
 	(segment
@@
 		(width 0.2)
 		(layer "F.Cu")
-		(net 12)
+		(net 11)
 	)
 	(segment
@@
 		(width 0.2)
 		(layer "F.Cu")
-		(net 12)
+		(net 11)
+	)
+	(segment
+		(start 74.911999 67.564)
+		(end 74.362 67.564)
+		(width 0.2)
+		(layer "F.Cu")
+		(net 11)
 	)
 	(segment
@@
 		(width 0.2)
 		(layer "F.Cu")
-		(net 12)
+		(net 11)
+	)
+	(segment
+		(start 76.854968 68.165)
+		(end 75.512999 68.165)
+		(width 0.2)
+		(layer "F.Cu")
+		(net 11)
 	)
 	(segment
@@
 		(width 0.2)
 		(layer "F.Cu")
-		(net 12)
+		(net 11)
 	)
 	(segment
@@
 		(width 0.2)
 		(layer "F.Cu")
-		(net 12)
+		(net 11)
 	)
 	(segment
@@
 		(width 0.2)
 		(layer "F.Cu")
-		(net 12)
+		(net 11)
 	)
 	(segment
@@
 		(width 0.2)
 		(layer "F.Cu")
-		(net 12)
+		(net 11)
 	)
 	(segment
@@
 		(width 0.2)
 		(layer "F.Cu")
-		(net 12)
+		(net 11)
 	)
 	(segment
@@
 		(width 0.2)
 		(layer "F.Cu")
-		(net 12)
+		(net 11)
 	)
 	(segment
@@
 		(width 0.2)
 		(layer "F.Cu")
-		(net 12)
+		(net 11)
 	)
 	(segment
@@
 		(width 0.2)
 		(layer "F.Cu")
-		(net 12)
+		(net 11)
 	)
 	(segment
@@
 		(width 0.2)
 		(layer "F.Cu")
-		(net 12)
+		(net 11)
 	)
 	(segment
@@
 		(width 0.2)
 		(layer "F.Cu")
-		(net 12)
+		(net 11)
 	)
 	(segment
@@
 		(width 0.2)
 		(layer "F.Cu")
-		(net 12)
+		(net 11)
 	)
 	(segment
@@
 		(width 0.2)
 		(layer "F.Cu")
-		(net 12)
+		(net 11)
+	)
+	(segment
+		(start 77.813 74.6535)
+		(end 77.813 69.123032)
+		(width 0.2)
+		(layer "F.Cu")
+		(net 11)
 	)
 	(segment
@@
 		(width 0.2)
 		(layer "F.Cu")
-		(net 12)
+		(net 11)
 	)
 	(zone
