File: 02 - Documentation/MODAC/Cartes Elec/Temp_Sensor_Cx/Temp_Sensor_Circuit_Side2/Temp_Sensor_Circuit_Side2.kicad_sch (KiCad schematic)
At the start: 9 parts, among them J1 Conn_01x09_Pin

Commit message: pcb_therm
Parts:
- removed J1: Conn_01x09_Pin, 5-1049359:51049359, symbol Connector:Conn_01x09_Pin
- added J2: Conn_01x09_Pin, Connector_PinHeader_1.27mm:PinHeader_1x09_P1.27mm_Vertical_SMD_Pin1Left, symbol Connector:Conn_01x09_Pin
- U1, U3, U4, U5, U6, U7, U8: footprint EPSA_lib:NTC_B3380 -> therm2:therm
- U2: footprint EPSA_lib:NTC_B3380 -> therm:therm
Connections:
- net GND: now also J2.1 (Pin_1)
- net at U6.1: now also J2.4 (Pin_4)
- net at U3.1: now also J2.7 (Pin_7)
- net at U8.1: now also J2.2 (Pin_2)
- net at U5.1: now also J2.5 (Pin_5)
- net at U1.1: now also J2.9 (Pin_9)
- net at U4.1: now also J2.6 (Pin_6)
- net at U2.1: now also J2.8 (Pin_8)
- net at U7.1: now also J2.3 (Pin_3)
Changed lines of the file:
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@@
 	)
 	(junction
-		(at 144.5177 105.2077)
+		(at 147.32 105.2077)
 		(diameter 0)
 		(color 0 0 0 0)
@@
 	(wire
 		(pts
-			(xy 126.6805 106.68) (xy 126.6805 89.4477)
-		)
-		(stroke
-			(width 0)
-			(type default)
-		)
-	)
-	(wire
-		(pts
-			(xy 118.8028 84.3677) (xy 144.5177 84.3677)
+			(xy 147.32 105.2077) (xy 144.5177 105.2077)
+		)
+		(stroke
+			(width 0)
+			(type default)
+		)
+	)
+	(wire
+		(pts
+			(xy 126.6805 106.68) (xy 126.6805 90.17)
+		)
+		(stroke
+			(width 0)
+			(type default)
+		)
+	)
+	(wire
+		(pts
+			(xy 118.8028 85.09) (xy 147.32 85.09)
 		)
 		(stroke
@@
 	(wire
 		(pts
-			(xy 118.8028 87.63) (xy 118.8028 84.3677)
+			(xy 118.8028 87.63) (xy 118.8028 85.09)
 		)
 		(stroke
@@
 	(wire
 		(pts
-			(xy 144.5177 105.2077) (xy 153.6479 105.2077)
-		)
-		(stroke
-			(width 0)
-			(type default)
-		)
-	)
-	(wire
-		(pts
 			(xy 144.5177 105.2077) (xy 144.5177 132.7421)
 		)
@@
 	(wire
 		(pts
-			(xy 129.6347 79.2877) (xy 144.5177 79.2877)
-		)
-		(stroke
-			(width 0)
-			(type default)
-		)
-	)
-	(wire
-		(pts
-			(xy 144.5177 97.0677) (xy 144.5177 105.2077)
+			(xy 129.6347 80.01) (xy 147.32 80.01)
+		)
+		(stroke
+			(width 0)
+			(type default)
+		)
+	)
+	(wire
+		(pts
+			(xy 147.32 97.79) (xy 147.32 105.2077)
 		)
 		(stroke
@@
 	(wire
 		(pts
-			(xy 135.364 76.7477) (xy 144.5177 76.7477)
+			(xy 135.364 77.47) (xy 147.32 77.47)
 		)
 		(stroke
@@
 	(wire
 		(pts
-			(xy 125.5168 81.8277) (xy 144.5177 81.8277)
-		)
-		(stroke
-			(width 0)
-			(type default)
-		)
-	)
-	(wire
-		(pts
-			(xy 132.947 91.9877) (xy 144.5177 91.9877)
-		)
-		(stroke
-			(width 0)
-			(type default)
-		)
-	)
-	(wire
-		(pts
-			(xy 137.5125 94.5277) (xy 144.5177 94.5277)
+			(xy 125.5168 82.55) (xy 147.32 82.55)
+		)
+		(stroke
+			(width 0)
+			(type default)
+		)
+	)
+	(wire
+		(pts
+			(xy 132.947 92.71) (xy 147.32 92.71)
+		)
+		(stroke
+			(width 0)
+			(type default)
+		)
+	)
+	(wire
+		(pts
+			(xy 137.5125 95.25) (xy 147.32 95.25)
 		)
 		(stroke
@@
 	(wire
 		(pts
-			(xy 126.6805 89.4477) (xy 144.5177 89.4477)
-		)
-		(stroke
-			(width 0)
-			(type default)
-		)
-	)
-	(wire
-		(pts
-			(xy 122.5626 86.9077) (xy 144.5177 86.9077)
-		)
-		(stroke
-			(width 0)
-			(type default)
-		)
-	)
-	(wire
-		(pts
-			(xy 125.5168 77.47) (xy 125.5168 81.8277)
+			(xy 126.6805 90.17) (xy 147.32 90.17)
+		)
+		(stroke
+			(width 0)
+			(type default)
+		)
+	)
+	(wire
+		(pts
+			(xy 122.5626 87.63) (xy 147.32 87.63)
+		)
+		(stroke
+			(width 0)
+			(type default)
+		)
+	)
+	(wire
+		(pts
+			(xy 125.5168 77.47) (xy 125.5168 82.55)
 		)
 		(stroke
@@
 	(wire
 		(pts
-			(xy 129.6347 68.58) (xy 129.6347 79.2877)
-		)
-		(stroke
-			(width 0)
-			(type default)
-		)
-	)
-	(wire
-		(pts
-			(xy 135.364 58.42) (xy 135.364 76.7477)
-		)
-		(stroke
-			(width 0)
-			(type default)
-		)
-	)
-	(wire
-		(pts
-			(xy 122.5626 96.52) (xy 122.5626 86.9077)
-		)
-		(stroke
-			(width 0)
-			(type default)
-		)
-	)
-	(wire
-		(pts
-			(xy 132.947 116.84) (xy 132.947 91.9877)
+			(xy 129.6347 68.58) (xy 129.6347 80.01)
+		)
+		(stroke
+			(width 0)
+			(type default)
+		)
+	)
+	(wire
+		(pts
+			(xy 135.364 58.42) (xy 135.364 77.47)
+		)
+		(stroke
+			(width 0)
+			(type default)
+		)
+	)
+	(wire
+		(pts
+			(xy 122.5626 96.52) (xy 122.5626 87.63)
+		)
+		(stroke
+			(width 0)
+			(type default)
+		)
+	)
+	(wire
+		(pts
+			(xy 132.947 116.84) (xy 132.947 92.71)
+		)
+		(stroke
+			(width 0)
+			(type default)
+		)
+	)
+	(wire
+		(pts
+			(xy 147.32 105.2077) (xy 153.6479 105.2077)
 		)
 		(stroke
@@
 	(wire
 		(pts
-			(xy 137.5125 127.0838) (xy 137.5125 94.5277)
+			(xy 137.5125 127.0838) (xy 137.5125 95.25)
 		)
 		(stroke
@@
 			(width 0)
 			(type default)
+		)
+	)
+	(symbol
+		(lib_id "Connector:Conn_01x09_Pin")
+		(at 152.4 87.63 180)
+		(unit 1)
+		(exclude_from_sim no)
+		(in_bom yes)
+		(on_board yes)
+		(dnp no)
+		(property "Reference" "J2"
+			(at 151.765 102.87 0)
+			(effects
+				(font
+					(size 1.27 1.27)
+				)
+			)
+		)
+		(property "Value" "Conn_01x09_Pin"
+			(at 151.765 100.33 0)
+			(effects
+				(font
+					(size 1.27 1.27)
+				)
+			)
+		)
+		(property "Footprint" "Connector_PinHeader_1.27mm:PinHeader_1x09_P1.27mm_Vertical_SMD_Pin1Left"
+			(at 166.624 83.82 0)
+			(effects
+				(font
+					(size 1.27 1.27)
+				)
+				(hide yes)
+			)
+		)
+		(property "Datasheet" "~"
+			(at 152.4 87.63 0)
+			(effects
+				(font
+					(size 1.27 1.27)
+				)
+				(hide yes)
+			)
+		)
+		(property "Description" "Generic connector, single row, 01x09, script generated"
+			(at 152.4 87.63 0)
+			(effects
+				(font
+					(size 1.27 1.27)
+				)
+				(hide yes)
+			)
+		)
+		(pin "5"
+		)
+		(pin "4"
+		)
+		(pin "7"
+		)
+		(pin "8"
+		)
+		(pin "9"
+		)
+		(pin "6"
+		)
+		(pin "1"
+		)
+		(pin "2"
+		)
+		(pin "3"
+		)
+		(instances
+			(project ""
+				(path "/706ac685-deb1-495b-9eb2-05b5f41532cb"
+					(reference "J2")
+					(unit 1)
+				)
+			)
 		)
 	)
@@
 			)
 		)
-		(property "Footprint" "EPSA_lib:NTC_B3380"
+		(property "Footprint" "therm2:therm"
 			(at 101.6 102.87 0)
 			(effects
@@
 			)
 		)
-		(property "Footprint" "EPSA_lib:NTC_B3380"
+		(property "Footprint" "therm2:therm"
 			(at 101.6 73.66 0)
 			(effects
@@
 			)
 		)
-		(property "Footprint" "EPSA_lib:NTC_B3380"
+		(property "Footprint" "therm2:therm"
 			(at 101.8408 123.2738 0)
 			(effects
@@
 			)
 		)
-		(property "Footprint" "EPSA_lib:NTC_B3380"
+		(property "Footprint" "therm2:therm"
 			(at 101.6 92.71 0)
 			(effects
@@
 			)
 		)
-		(property "Footprint" "EPSA_lib:NTC_B3380"
+		(property "Footprint" "therm2:therm"
 			(at 101.6 54.61 0)
 			(effects
@@
 			)
 		)
-		(property "Footprint" "EPSA_lib:NTC_B3380"
+		(property "Footprint" "therm2:therm"
 			(at 101.6 83.82 0)
 			(effects
@@
 			)
 		)
-		(property "Footprint" "EPSA_lib:NTC_B3380"
+		(property "Footprint" "therm:therm"
 			(at 101.6 64.77 0)
 			(effects
@@
 			)
 		)
-		(property "Footprint" "EPSA_lib:NTC_B3380"
+		(property "Footprint" "therm2:therm"
 			(at 101.6 113.03 0)
 			(effects
@@
 					(unit 1)
 				)
-			)
-		)
-	)
-	(symbol
-		(lib_id "Connector:Conn_01x09_Pin")
-		(at 149.5977 86.9077 180)
-		(unit 1)
-		(exclude_from_sim no)
-		(in_bom yes)
-		(on_board yes)
-		(dnp no)
-		(fields_autoplaced yes)
-		(property "Reference" "J1"
-			(at 151.13 85.6376 0)
-			(effects
-				(font
-					(size 1.27 1.27)
-				)
-				(justify right)
-			)
-		)
-		(property "Value" "Conn_01x09_Pin"
-			(at 151.13 88.1776 0)
-			(effects
-				(font
-					(size 1.27 1.27)
-				)
-				(justify right)
-			)
-		)
-		(property "Footprint" "5-1049359:51049359"
-			(at 149.5977 86.9077 0)
-			(effects
-				(font
-					(size 1.27 1.27)
-				)
-				(hide yes)
-			)
-		)
-		(property "Datasheet" "~"
-			(at 149.5977 86.9077 0)
-			(effects
-				(font
-					(size 1.27 1.27)
-				)
-				(hide yes)
-			)
-		)
-		(property "Description" "Generic connector, single row, 01x09, script generated"
-			(at 149.5977 86.9077 0)
-			(effects
-				(font
-					(size 1.27 1.27)
-				)
-				(hide yes)
-			)
-		)
-		(pin "1"
-		)
-		(pin "2"
-		)
-		(pin "4"
-		)
-		(pin "3"
-		)
-		(pin "6"
-		)
-		(pin "5"
-		)
-		(pin "7"
-		)
-		(pin "8"
-		)
-		(pin "9"
-		)
-		(instances
-			(project ""
-				(path "/706ac685-deb1-495b-9eb2-05b5f41532cb"
-					(reference "J1")
-					(unit 1)
-				)

Commit message: dernière version temps sensors
Parts:
- J2: footprint Connector_PinHeader_1.27mm:PinHeader_1x09_P1.27mm_Vertical_SMD_Pin1Left -> Connector_PinHeader_2.54mm:PinHeader_1x09_P2.54mm_Vertical_SMD_Pin1Left
Changed lines of the file:
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@@
 			)
 		)
-		(property "Footprint" "Connector_PinHeader_1.27mm:PinHeader_1x09_P1.27mm_Vertical_SMD_Pin1Left"
+		(property "Footprint" "Connector_PinHeader_2.54mm:PinHeader_1x09_P2.54mm_Vertical_SMD_Pin1Left"
 			(at 166.624 83.82 0)
 			(effects
