File: 02 - Documentation/BASTIE/Cartes Artemiz/BSPD_v4/bspdv4.kicad_pcb (KiCad board)
At the start: 2 copper layers, 89.8 x 62.2 mm, 65 parts, among them J1 3P Droit 22-11-2032, J2 3P Droit 22-11-2032, J3 2P Droit 2-11-2022, J4 2P Droit 2-11-2022, K1 SSR CPC1394GR, K2 SSR CPC1394GR, Q1 PMOS SI2343CDS-T1-GE3, U2 Alim LP TSR_0.5-2450

Commit message: BSPD v4 / AMS IMD v3
Parts:
- moved H2 208.6 mm to (235.9, 82.1)
- moved C5 182.3 mm to (226.0, 81.3)
- moved R12 165.3 mm to (205.8, 68.0), turned to 0 degrees
- moved TP3 163.3 mm to (235.3, 57.8)
- moved R7 163.2 mm to (230.1, 77.2), turned to 180 degrees
- moved J3 162.6 mm to (234.7, 47.8), turned to -90 degrees
- moved C2 159.2 mm to (236.9, 69.7)
- moved G4 159.0 mm to (224.9, 75.2)
- moved G2 157.0 mm to (218.1, 63.7), turned to 90 degrees
- moved TP4 157.0 mm to (235.4, 54.5)
- moved K2 156.6 mm to (223.9, 45.7)
- moved CP3 155.9 mm to (228.2, 69.8), turned to 180 degrees
- moved H3 155.1 mm to (184.7, 40.1)
- moved TP6 154.8 mm to (208.9, 45.5)
- moved R3 154.7 mm to (233.1, 67.2), turned to 90 degrees
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Routing:
- net +5V: track 42.2 -> 293.6 mm, vias 22 -> 3
- net SCS Check: track 101.3 -> 68.4 mm
- net 4.25V: track 14.6 -> 36.8 mm, vias 0 -> 3
- net 0.75V: track 19.4 -> 40.1 mm, vias 2 -> 4
- net GND: track 0.00 -> 16.8 mm, vias 0 -> 8
- net Net-(CP3-IN-): track 24.5 -> 9.74 mm
- net Net-(CP1-OUT): track 63.9 -> 50.5 mm, vias 1 -> 2
- net +12V: track 28.9 -> 17.0 mm
- net Intput w/ 50msdelay: track 73.6 -> 62.6 mm, vias 2 -> 1
- net Net-(G4-Pad4): track 3.33 -> 13.4 mm
- net Net-(CP2-OUT): track 62.3 -> 52.3 mm
- net Net-(G2-Pad4): track 32.8 -> 23.2 mm
- net Raw Current Sensor: track 11.0 -> 19.9 mm
- net SC in: track 16.1 -> 7.78 mm
- net BSPD out: track 57.1 -> 49.0 mm
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- added copper zone on B.Cu, net GND
- removed copper zone on B.Cu, net +5V
Other:
- board size 89.8 x 62.2 mm -> 77.3 x 55.8 mm
- board text added: "CS+BPS"
- board text added: "Current"
- board text added: "GND 12V"
- board text removed: "12V|GND"
- board text removed: "CS+BPS w/50ms"
- board text removed: "Current sensor"
