File: 02 - Documentation/BASTIE/Cartes Artemiz/JLCPCB-ver/SCS IMD-AMD-indicator/SCS IMD-AMD-indicator.kicad_sch (KiCad schematic)
At the start: 23 parts, among them J1 Conn_01x02, J2 Conn_01x02, U1 LM393DR2G, U2 74AHC1G32, U3 74AHC1G00, U4 CPC1017N, U5 LMV321IDBVR, U6 78L05G, U7 LMV321IDBVR, U8 LMV321IDBVR

Commit message: corrections jlcp ver cartes
Connections:
- net PCB_State_OK: now also U5.1 (+), U7.3 (-), U7.4 (OUT), U8.3 (-)
Changed lines of the file:
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@@
+		)
+	)
+	(label "PCB_State_OK"
+		(at 82.55 137.16 0)
+		(effects
+			(font
+				(size 1.27 1.27)
+			)
+			(justify left bottom)
 		)
 	)

Commit message: MAJ cartes électroniques
Parts:
- C1: Price 0.026USD -> 0.029USD; Stock 3458747 -> 1168756
- C2: Price 0.016USD -> 0.015USD; Stock 27578 -> 92471
- C3: Stock 8754636 -> 5698112
- R1, R5: Stock 29702 -> 182449
- R10: Stock 93506 -> 272497
- R2, R9: Stock 14905033 -> 6826120
- R3, R7: Stock 60670 -> 91172
- R4, R6: Stock 212769 -> 276235
- R8: Stock 877100 -> 1203703
- U1: Stock 236587 -> 198289
- U5, U7, U8: Price 0.103USD -> 0.075USD; Stock 119521 -> 138487
- U6: Stock 84902 -> 62898
Connections:
- no-connect marks 1 -> 3
